File: hardware/connected_sensor.sch (KiCad schematic (older format))
At the start: 43 parts, among them J1 Conn_01x04, J2 Conn_01x04, J3 Conn_01x05, J4 Conn_01x05, J5 Conn_01x03, J6 AC_IN, J7 LOAD, J8 UEXT, K1 G2RL-1A-E 5DC, M1 ESP8266-DEV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

Commit message: L'ecran necessite 2 GPIOs en plus du SPI. Re-route 2 GPIOs de l'ESP vers le connecteur ecran.
Parts:
- C1, C2, C3, C4, C5, C6: symbol C_Small -> connected_sensor-rescue:C_Small
- D1: symbol D_Small -> connected_sensor-rescue:D_Small
- J1, J2: symbol Conn_01x04 -> connected_sensor-rescue:Conn_01x04
- J3, J4: symbol Conn_01x05 -> connected_sensor-rescue:Conn_01x05
- J5: symbol Conn_01x03 -> connected_sensor-rescue:Conn_01x03
- J6, J7: symbol Conn_01x02 -> connected_sensor-rescue:Conn_01x02
- J8: symbol Conn_02x05_Odd_Even -> connected_sensor-rescue:Conn_02x05_Odd_Even
- K1: symbol RM50-xx21 -> connected_sensor-rescue:RM50-xx21
- M1: symbol ESP8266-DEV -> connected_sensor-rescue:ESP8266-DEV
- Q1: symbol Q_NMOS_GDS -> connected_sensor-rescue:Q_NMOS_GSD
- R1, R10, R11, R12, R13, R14, R15, R2, R3, R4, R5, R6, R7, R8, R9: symbol R_Small -> connected_sensor-rescue:R_Small
- SW1, SW2, SW3, SW4: symbol SW_Push -> connected_sensor-rescue:SW_Push
- SW5: symbol 5G -> connected_sensor-rescue:5G
- T1: symbol Transformer_1P_1S -> connected_sensor-rescue:Transformer_1P_1S
- U1: symbol MAX4460ESA -> connected_sensor-rescue:MAX4460ESA
- U2: symbol PIC18F25Q10 -> connected_sensor-rescue:PIC18F25Q10
- U3: symbol IRM-03 -> connected_sensor-rescue:IRM-03
- U4: symbol MIC5205-3.3 -> connected_sensor-rescue:MIC5205-3.3
Connections:
- net labels added: C_D, LCD_RST
- wire segments 167 -> 212
Other:
- moved on the sheet: D1, K1, Q1, R12, R13, R8
