File: hardware/connected_sensor.kicad_pcb (KiCad board)
At the start: 2 copper layers, 110 x 70 mm, 42 parts, among them J1 Conn_01x04, J2 Conn_01x04, J3 Conn_01x05, J4 Conn_01x05, J5 Conn_01x03, J6 AC_IN, J7 LOAD, J8 UEXT, K1 G2RL-1A-E 5DC, M1 ESP8266-DEV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

Commit message: L'ecran necessite 2 GPIOs en plus du SPI. Re-route 2 GPIOs de l'ESP vers le connecteur ecran.
Parts:
- moved R12 76.1 mm to (105.0, 125.1), turned to 0 degrees
- moved R13 7.62 mm to (87.0, 57.1), turned to 90 degrees
- moved Q1 1.42 mm to (100.3, 76.8), turned to 310 degrees
Connections:
- J8 pad 5: SCL -> /LCD_RST
- J8 pad 6: SDA -> /C_D
- M1 pad 11: REL -> /LCD_RST
- M1 pad 21: Net-(M1-Pad21) -> /C_D
- Q1 pad 1: REL -> /REL
- Q1 pad 2: Net-(D1-Pad2) -> GND
- Q1 pad 3: GND -> Net-(D1-Pad2)
- R12 pad 1: +3V3 -> SDA
- R12 pad 2: SDA -> +3V3
- R13 pad 1: +3V3 -> SCL
- R13 pad 2: SCL -> +3V3
- R15 pad 2: Net-(M1-Pad21) -> /C_D
- R8 pad 1: REL -> /REL
- U1 pad 4: Net-(C1-Pad1) -> (no net)
- U1 pad 5: Net-(R2-Pad1) -> (no net)
- U1 pad 6: +3V3 -> Net-(C1-Pad1)
- U2 pad 18: REL -> /REL
Routing:
- net REL: track 162.2 -> 0.00 mm
- net /REL: track 0.00 -> 154.6 mm
- net /C_D: track 0.00 -> 40.3 mm, vias 0 -> 2
- net /LCD_RST: track 0.00 -> 38.5 mm, vias 0 -> 1
- net SDA: track 103.0 -> 72.2 mm, vias 4 -> 2
- net Net-(M1-Pad21): track 9.04 -> 0.00 mm
- net SCL: track 89.2 -> 86.0 mm
- net +3V3: track 181.6 -> 179.5 mm
- net Net-(C1-Pad1): track 6.49 -> 8.56 mm

Commit message: Convert to kicad 6.x
Other:
- net class AC removed
- net class Default removed
