File: hardware/max4460_fix.kicad_pcb (KiCad board)
At the start: 2 copper layers, 21.6 x 19 mm, 8 parts, among them J1 Conn_01x04, J2 Conn_01x04, J3 Conn_01x01, U1 MAX4460ESA

Commit message: Convert to kicad 6.x
Other:
- net class AC removed
- net class Default removed
